File: CAN Toolboard redesign/CAN_toolboard_redesign.brd (EAGLE design)
At the start: 49 x 54.2 mm, 142 parts, among them J3 430450400CON_430450400_MOL, M1 NMOSFET_WSD3066DN33, M2 CJ3400, M3 CJ3400, M4 CJ3400, P1 TPS54202_BUCKCONV, P2 3.3V, U1 RP2040IC57_RP2040-L, U2 W25Q128JVSIQSOIC_128JVSIQ_WIN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, U3 SN65HVD1050DRD8-L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

Commit message: Updated as of 05/08/23
Parts:
- moved D4 61.6 mm to (25.3, 52.5), turned to 180 degrees
- moved M3 58.8 mm to (65.5, 61.2), turned to 180 degrees
- moved R46 57.9 mm to (65.5, 58.2), turned to 90 degrees
- moved R47 52.8 mm to (64.2, 58.2), turned to 90 degrees
- moved D7 51.6 mm to (57.5, 59.5)
- moved R35 42.1 mm to (38.8, 44.8), turned to 180 degrees
- moved R44 36.3 mm to (48.2, 35.3), turned to 180 degrees
- moved D6 35.4 mm to (48.2, 40.1), turned to 90 degrees
- moved R33 35.2 mm to (42.7, 44.1)
- moved C40 34.2 mm to (55.4, 35.8), turned to 180 degrees
- moved R40 33.5 mm to (48.2, 48.8), turned to 180 degrees
- moved R45 33.3 mm to (50.0, 33.9), turned to 180 degrees
- moved M4 33.0 mm to (40.6, 31.9), turned to 90 degrees
- moved D8 31.9 mm to (40.7, 28.5), turned to 90 degrees
- moved R36 31.7 mm to (54.7, 36.8)
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Connections:
- net CAN_N: now also X2.1; no longer X2.2
- net CAN_P: now also X2.2; no longer X2.1
Routing:
- net +3.3V: track 1.37 -> 71.2 mm, vias 0 -> 7
- net FAN2: track 0.00 -> 39.6 mm, vias 0 -> 4
- net HE0: track 0.00 -> 38.7 mm, vias 0 -> 4
- net QSPI_SD0: track 0.00 -> 25.8 mm, vias 0 -> 2
- net SPI1_MOSI: track 0.00 -> 25.8 mm, vias 0 -> 2
- net QSPI_SD3: track 0.00 -> 25.3 mm, vias 0 -> 2
- net SPI1_SCK: track 0.00 -> 25.2 mm, vias 0 -> 2
- net QSPI_SCK: track 0.00 -> 23.8 mm, vias 0 -> 2
- net QSPI_SS: track 0.00 -> 22.6 mm, vias 0 -> 2
- net QSPI_SD1: track 0.00 -> 21.5 mm, vias 0 -> 2
- net SPI1_MISO: track 0.00 -> 20.4 mm, vias 0 -> 2
- net QSPI_SD2: track 0.00 -> 20.3 mm, vias 0 -> 2
- net E0_DIR: track 0.00 -> 19.2 mm, vias 0 -> 2
- net LED: track 0.00 -> 18.6 mm, vias 0 -> 2
- net FAN1G: track 0.00 -> 17.6 mm, vias 0 -> 2
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
Commit message: updated as of 07.08.23
Parts:
- removed IO1, IO2, IO3: TEST-POINT3, SparkFun-Connectors:PAD.03X.03
- removed TH0: TEST-POINT3X4, SparkFun-Connectors:PAD.03X.04
- added TH0A, USB1_N, USB1_P: TEST-POINT3X4, SparkFun-Connectors:PAD.03X.04
- moved GND 73.6 mm to (30.4, 63.7)
- moved A2 43.1 mm to (46.3, 13.8)
- moved A1 43.0 mm to (49.0, 13.7)
- moved HE0 36.4 mm to (25.2, 36.2), flipped to the bottom
- moved B1 35.4 mm to (51.6, 13.8)
- moved 5V 31.7 mm to (35.5, 64.1)
- moved B2 30.5 mm to (54.0, 13.8)
- moved 24V 26.2 mm to (37.1, 64.2)
- moved 3.3V 20.3 mm to (33.9, 64.1)
- moved R15 1.40 mm to (35.1, 18.9)
- moved C14 1.27 mm to (35.1, 20.3)
- moved D3 1.15 mm to (35.0, 17.3)
- moved C32 1.02 mm to (52.4, 34.1)
- moved C17 1.02 mm to (35.0, 21.6)
- moved C11 0.69 mm to (49.6, 42.1)
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Connections:
- net +5V: no longer IO3.P$1
- net TH0: no longer TH0.P$1
- net TH0A: now also TH0A.P$1
- net USB1_N: now also USB1_N.P$1
- net USB1_P: now also USB1_P.P$1
- net USB_N: no longer IO1.P$1
- net USB_P: no longer IO2.P$1
Routing:
- net GND: track 4.32 -> 400.2 mm, vias 18 -> 54
- net +3.3V: track 71.2 -> 261.3 mm, vias 7 -> 28
- net FAN0: track 1.71 -> 133.3 mm, vias 1 -> 8
- net +5V: track 11.1 -> 140.1 mm, vias 2 -> 12
- net TH0B: track 0.00 -> 100.8 mm, vias 0 -> 7
- net N$1: track 0.00 -> 56.6 mm, vias 0 -> 3
- net N$2: track 0.00 -> 53.4 mm, vias 0 -> 2
- net +24V: track 101.1 -> 135.6 mm
- net TH0A: track 0.00 -> 29.3 mm, vias 0 -> 2
- net RESET: track 0.00 -> 26.9 mm, vias 0 -> 2
- net VBUS: track 4.93 -> 31.3 mm, vias 0 -> 2
- net +1.1V: track 13.3 -> 38.6 mm, vias 2 -> 5
- net FAN1: track 3.89 -> 28.2 mm, vias 1 -> 4
- net XR: track 0.00 -> 23.6 mm, vias 0 -> 4
- net HE0_PWR: track 0.00 -> 20.2 mm, vias 0 -> 4
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- added copper zone on layer 1, net HE0_PWR
- added copper zone on layer 16, net HE0_PWR
Other:
- outline, holes or cut-outs redrawn
