File: CAN Toolboard redesign/CAN_toolboard_redesign.brd (EAGLE design)
At the start: 49 x 54.2 mm, 142 parts, among them J3 430450400CON_430450400_MOL, M1 NMOSFET_WSD3066DN33, M2 CJ3400, M3 CJ3400, M4 CJ3400, P1 TPS54202_BUCKCONV, P2 3.3V, U1 RP2040IC57_RP2040-L, U2 W25Q128JVSIQSOIC_128JVSIQ_WIN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, U3 SN65HVD1050DRD8-L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

Commit message: updated board as of 04/08/23
Parts:
- moved C17 65.0 mm to (37.1, 20.2)
- moved C14 64.7 mm to (33.8, 20.3)
- moved R15 63.9 mm to (33.7, 19.0), turned to 180 degrees
- moved C15 62.2 mm to (36.3, 17.6), turned to 90 degrees
- moved C16 61.0 mm to (26.6, 23.5)
- moved P2 60.6 mm to (30.1, 18.8), turned to 180 degrees
- moved D3 58.8 mm to (33.8, 17.2)
- moved L2 58.3 mm to (53.5, 56.2), turned to 180 degrees
- moved R3 51.4 mm to (44.0, 38.3), turned to 90 degrees
- moved R4 51.1 mm to (42.7, 38.3), turned to 270 degrees
- moved U3 50.8 mm to (55.0, 52.0), turned to 90 degrees
- moved C27 50.7 mm to (50.4, 48.9), turned to 180 degrees
- moved X1 50.3 mm to (55.7, 46.4)
- moved C26 49.4 mm to (57.1, 56.3)
- moved C4 47.9 mm to (55.1, 43.0)
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Routing:
- net VREGO: track 16.5 -> 0.00 mm, vias 2 -> 0
- net +24V: track 88.5 -> 102.5 mm, vias 6 -> 7
- net TMCENN: track 0.00 -> 12.5 mm
- net A2: track 0.00 -> 11.2 mm, vias 0 -> 1
- net +5V: track 0.00 -> 11.1 mm, vias 0 -> 2
- net B2: track 0.00 -> 10.7 mm
- net A1: track 0.00 -> 8.90 mm
- net B1: track 0.00 -> 8.84 mm
- net DIR: track 0.00 -> 5.23 mm
- net VREGFB: track 0.00 -> 4.93 mm
- net TMC5V: track 0.00 -> 4.59 mm
- net E0_UART: track 0.00 -> 4.02 mm
- net VRC: track 0.00 -> 3.57 mm
- net STEP: track 0.00 -> 3.41 mm
- net BRA: track 0.00 -> 2.98 mm
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
Commit message: Created New Schematic
Parts:
- moved C33 6.93 mm to (40.6, 18.8)
- moved C15 4.96 mm to (36.6, 22.6)
- moved C14 4.84 mm to (38.0, 22.6), turned to 90 degrees
- moved C17 3.05 mm to (35.1, 22.6), turned to 90 degrees
Routing:
- net +24V: track 102.5 -> 7.53 mm
- net A2: track 11.2 -> 0.00 mm, vias 1 -> 0
- net B2: track 10.7 -> 0.54 mm
- net A1: track 8.90 -> 0.00 mm
- net B1: track 8.84 -> 0.00 mm
- net +5V: track 11.1 -> 5.25 mm, vias 2 -> 0
- net VRC: track 3.57 -> 0.00 mm
- net VREGFB: track 4.93 -> 2.18 mm
- net VREGEN: track 2.69 -> 0.00 mm
