File: CAN Toolboard redesign/CAN_toolboard_redesign.sch (EAGLE design)
At the start: 151 parts, among them J2 2828XX-2282837-2, J3 430450400CON_430450400_MOL, M1 NMOSFET_WSD3066DN33, M2 CJ3400, M3 CJ3400, M4 CJ3400, P1 TPS54202_BUCKCONV, P2 3.3V, U1 RP2040IC57_RP2040-L, U2 W25Q128JVSIQSOIC_128JVSIQ_WIN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

Commit message: Added eagle files for current progress in toolboard
Parts:
- removed 120R, PT1000, VBUS: PINHD-1X2, Fracktal Misc Lib:PINHD-1X2
- removed C41: 1uF, Fracktal Misc Lib:C_CHIP-0402(1005-METRIC)
- removed C46: 10uF, Fracktal Misc Lib:C_CHIP-0603(1608-METRIC)
- removed D5: BAT54S, Fracktal Misc Lib:BAT54S
- removed IO16, IO17, IO18, IO19, IO22, IO23: TEST-POINT3, SparkFun-Connectors:TEST-POINT3
- removed J2: 2828XX-2282837-2, Connector:2828XX-2282837-2
- removed R32: 120R, Fracktal Misc Lib:R_CHIP-0402(1005-METRIC)
- removed R38: 10K, Fracktal Misc Lib:R_CHIP-0402(1005-METRIC)
- removed RGB, SERVO: PINHD-1X3, Fracktal Misc Lib:PINHD-1X3
- removed SWCLK, SWDIO: TEST-POINT3X4, SparkFun-Connectors:TEST-POINT3X4
- removed TP1, TP3: TEST-POINT3, Fracktal Misc Lib:TEST-POINT3
- removed U4: SN74LVC1G17DBVRDBV5-L, 2023-03-28_15-41-49_Library:SN74LVC1G17DBVRDBV5-L
- added 24V, 3.3V, 5V, A1, A2, B1, B2, HE0, TH0: TEST-POINT3X4, SparkFun-Connectors:TEST-POINT3X4
- added J1: (no value), SparkFun-Connectors:CONN_023.5MM
- added SJ1, SJ3: SOLDERJUMPERTRACE, SparkFun-Retired:SOLDERJUMPERTRACE
- added SJ2: SOLDERJUMPERNO, SparkFun-Retired:SOLDERJUMPERNO
- X4: value JST-XH-02-PIN-LONG-PAD -> JST-XH-04-PIN-LONG-PAD; device Rembrandt Electronics - JST XH Connectors v1-0:JST-XH-02-PIN-LONG-PAD -> Rembrandt Electronics - JST XH Connectors v1-0:JST-XH-04-PIN-LONG-PAD
- X8: value JST-XH-04-PIN-LONG-PAD -> JST-XH-02-PIN-LONG-PAD; device Rembrandt Electronics - JST XH Connectors v1-0:JST-XH-04-PIN-LONG-PAD -> Rembrandt Electronics - JST XH Connectors v1-0:JST-XH-02-PIN-LONG-PAD
Connections:
- removed net FAN2D: M4.D, X4-1.S, X5-1.S
- removed net NEOPIXEL: R38.2, U1.GPIO3, U4.A
- removed net RGBDATA: R32.2, RGB.2
- removed net RGBDATA1: R32.1, U4.Y
- removed net SERVO: D5.3, SERVO.3, U1.GPIO11
- new net N$2: M4.D, X7-1.S, X8-1.S
- net +24V: now also 24V.1, J1.1, X6-2.S, X7-2.S, X8-2.S; no longer J2.1, X2-2.S, X3-2.S, X4-2.S
- net +3.3V: now also 3.3V.1, SJ2.2; no longer D5.2, PT1000.1, TP3.1
- net +5V: now also 5V.1; no longer C41.1, C46.2, RGB.1, SERVO.2, TP1.1, U4.VCC
- net A1: now also A1.1, X4-2.S; no longer X8-2.S
- net A2: now also A2.1, X4-1.S; no longer X8-1.S
- net B1: now also B1.1, X4-3.S; no longer X8-3.S
- net B2: now also B2.1, X4-4.S; no longer X8-4.S
- net CAN_N: now also SJ1.1, X2-2.S; no longer 120R.2, X7-2.S
- net CAN_P: now also X2-1.S; no longer X7-1.S
- net CNT: now also SJ1.2; no longer 120R.1
- net EX: now also X3-2.S; no longer X6-2.S
- net FAN1D: now also X6-1.S; no longer X3-1.S
- net GND: now also J1.2, X3-1.S; no longer C41.2, C46.1, D5.1, J2.2, R38.1, RGB.3, SERVO.1, U4.GND, X6-1.S
- net HE0: now also HE0.1
- net I2C_SCL: no longer IO23.1
- net I2C_SDA: no longer IO22.1
- net N$1: now also X5-1.S; no longer X2-1.S
- net SPI0_CS: no longer IO17.1
- net SPI0_MISO: no longer IO16.1
- net SPI0_MOSI: no longer IO19.1
- net SPI0_SCK: no longer IO18.1
- net SWCLK: no longer SWCLK.1
- net SWDIO: no longer SWDIO.1
- net TH0: now also TH0.1
- net TH0C: now also SJ2.1; no longer PT1000.2
- net VBUS: now also SJ3.2; no longer VBUS.2
- net VBUS1: now also SJ3.1; no longer VBUS.1
Other:
- note removed: "5.08mm Terminal Block"
- moved on the sheet: BOOT, C1, C10, C11, C12, C13, C14, C15, C16, C17, C18, C19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

Commit message: Updated as of 05/08/23
Connections:
- net CAN_N: now also X2-1.S; no longer X2-2.S
- net CAN_P: now also X2-2.S; no longer X2-1.S
Changed lines of the file:
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@@
 <net name="CAN_N" class="2">
-<segment>
-<label x="429.26" y="414.02" size="1.778" layer="95" xref="yes"/>
-<wire x1="429.26" y1="414.02" x2="414.02" y2="414.02" width="0.1524" layer="91"/>
-<wire x1="414.02" y1="414.02" x2="414.02" y2="411.48" width="0.1524" layer="91"/>
-<wire x1="414.02" y1="411.48" x2="383.54" y2="411.48" width="0.1524" layer="91"/>
-<pinref part="X2" gate="-2" pin="S"/>
-</segment>
 <segment>
 <wire x1="144.78" y1="256.54" x2="149.86" y2="256.54" width="0.1524" layer="91"/>
@@
 <pinref part="SJ1" gate="1" pin="1"/>
 <wire x1="144.78" y1="261.62" x2="170.18" y2="261.62" width="0.1524" layer="91"/>
+</segment>
+<segment>
+<pinref part="X2" gate="-1" pin="S"/>
+<wire x1="383.54" y1="408.94" x2="393.7" y2="408.94" width="0.1524" layer="91"/>
+<label x="393.7" y="408.94" size="1.778" layer="95"/>
 </segment>
 </net>
@@
 <net name="CAN_P" class="2">
 <segment>
-<label x="429.26" y="408.94" size="1.778" layer="95" xref="yes"/>
-<wire x1="429.26" y1="408.94" x2="383.54" y2="408.94" width="0.1524" layer="91"/>
-<pinref part="X2" gate="-1" pin="S"/>
-</segment>
-<segment>
 <wire x1="144.78" y1="281.94" x2="149.86" y2="281.94" width="0.1524" layer="91"/>
 <label x="149.86" y="281.94" size="1.27" layer="95" xref="yes"/>
@@
 <junction x="144.78" y="271.78"/>
 </segment>
+<segment>
+<pinref part="X2" gate="-2" pin="S"/>
+<wire x1="383.54" y1="411.48" x2="393.7" y2="411.48" width="0.1524" layer="91"/>
+<label x="393.7" y="411.48" size="1.778" layer="95"/>
+</segment>
 </net>

Commit message: updated as of 07.08.23
Parts:
- removed IO1, IO2, IO3: TEST-POINT3, SparkFun-Connectors:TEST-POINT3
- removed TH0: TEST-POINT3X4, SparkFun-Connectors:TEST-POINT3X4
- added TH0A, USB1_N, USB1_P: TEST-POINT3X4, SparkFun-Connectors:TEST-POINT3X4
Connections:
- net +5V: no longer IO3.1
- net TH0: no longer TH0.1
- net TH0A: now also TH0A.1
- net USB1_N: now also USB1_N.1
- net USB1_P: now also USB1_P.1
- net USB_N: no longer IO1.1
- net USB_P: no longer IO2.1
Changed lines of the file:
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@@
 <attribute name="LCSCPN#" value="C162274"/>
 </part>
-<part name="IO1" library="SparkFun-Connectors" library_urn="urn:adsk.eagle:library:513" deviceset="TEST-POINT" device="3" package3d_urn="urn:adsk.eagle:package:38286/1"/>
-<part name="IO2" library="SparkFun-Connectors" library_urn="urn:adsk.eagle:library:513" deviceset="TEST-POINT" device="3" package3d_urn="urn:adsk.eagle:package:38286/1"/>
-<part name="IO3" library="SparkFun-Connectors" library_urn="urn:adsk.eagle:library:513" deviceset="TEST-POINT" device="3" package3d_urn="urn:adsk.eagle:package:38286/1"/>
 <part name="SJ1" library="SparkFun-Retired" deviceset="SOLDERJUMPER" device="TRACE"/>
 <part name="SJ2" library="SparkFun-Retired" deviceset="SOLDERJUMPER" device="NO"/>
@@
 <part name="24V" library="SparkFun-Connectors" library_urn="urn:adsk.eagle:library:513" deviceset="TEST-POINT" device="3X4" package3d_urn="urn:adsk.eagle:package:38287/1"/>
 <part name="HE0" library="SparkFun-Connectors" library_urn="urn:adsk.eagle:library:513" deviceset="TEST-POINT" device="3X4" package3d_urn="urn:adsk.eagle:package:38287/1"/>
-<part name="TH0" library="SparkFun-Connectors" library_urn="urn:adsk.eagle:library:513" deviceset="TEST-POINT" device="3X4" package3d_urn="urn:adsk.eagle:package:38287/1"/>
 <part name="A2" library="SparkFun-Connectors" library_urn="urn:adsk.eagle:library:513" deviceset="TEST-POINT" device="3X4" package3d_urn="urn:adsk.eagle:package:38287/1"/>
 <part name="A1" library="SparkFun-Connectors" library_urn="urn:adsk.eagle:library:513" deviceset="TEST-POINT" device="3X4" package3d_urn="urn:adsk.eagle:package:38287/1"/>
@@
 <attribute name="FAN3" value=""/>
 </part>
+<part name="TH0A" library="SparkFun-Connectors" library_urn="urn:adsk.eagle:library:513" deviceset="TEST-POINT" device="3X4" package3d_urn="urn:adsk.eagle:package:38287/1"/>
+<part name="USB1_P" library="SparkFun-Connectors" library_urn="urn:adsk.eagle:library:513" deviceset="TEST-POINT" device="3X4" package3d_urn="urn:adsk.eagle:package:38287/1"/>
+<part name="USB1_N" library="SparkFun-Connectors" library_urn="urn:adsk.eagle:library:513" deviceset="TEST-POINT" device="3X4" package3d_urn="urn:adsk.eagle:package:38287/1"/>
 </parts>
 <sheets>
@@
 <attribute name="LCSCPN#" x="533.4" y="78.74" size="1.778" layer="96" display="off"/>
 </instance>
-<instance part="IO1" gate="G$1" x="386.08" y="313.436" smashed="yes" rot="R180">
-<attribute name="NAME" x="382.27" y="313.436" size="1.27" layer="95" font="vector" rot="R180" align="center-left"/>
-</instance>
-<instance part="IO2" gate="G$1" x="386.08" y="315.976" smashed="yes" rot="R180">
-<attribute name="NAME" x="382.27" y="315.976" size="1.27" layer="95" font="vector" rot="R180" align="center-left"/>
-</instance>
-<instance part="IO3" gate="G$1" x="396.24" y="326.136" smashed="yes" rot="R180">
-<attribute name="NAME" x="392.43" y="326.136" size="1.27" layer="95" font="vector" rot="R180" align="center-left"/>
-</instance>
 <instance part="SJ1" gate="1" x="170.18" y="266.7" smashed="yes" rot="R90">
 <attribute name="NAME" x="167.64" y="264.16" size="1.778" layer="95" rot="R90"/>
@@
 <instance part="HE0" gate="G$1" x="45.72" y="63.5" smashed="yes" rot="R180">
 <attribute name="NAME" x="40.64" y="63.5" size="1.778" layer="95" font="vector" rot="R180"/>
-</instance>
-<instance part="TH0" gate="G$1" x="447.04" y="238.76" smashed="yes">
-<attribute name="NAME" x="452.12" y="238.76" size="1.778" layer="95" font="vector"/>
 </instance>
 <instance part="A2" gate="G$1" x="391.16" y="182.88" smashed="yes">
@@
 <attribute name="VALUE" x="511.683" y="110.998" size="1.778" layer="96" rot="R90"/>
 <attribute name="FAN3" x="513.08" y="111.76" size="1.778" layer="96" rot="R90" display="name"/>
+</instance>
+<instance part="TH0A" gate="G$1" x="373.38" y="228.6" smashed="yes" rot="R180">
+<attribute name="NAME" x="368.3" y="228.6" size="1.778" layer="95" font="vector" rot="R180"/>
+</instance>
+<instance part="USB1_P" gate="G$1" x="497.84" y="314.96" smashed="yes">
+<attribute name="NAME" x="502.92" y="314.96" size="1.778" layer="95" font="vector"/>
+</instance>
+<instance part="USB1_N" gate="G$1" x="497.84" y="312.42" smashed="yes">
+<attribute name="NAME" x="502.92" y="312.42" size="1.778" layer="95" font="vector"/>
 </instance>
 </instances>
@@
 <wire x1="408.94" y1="314.96" x2="408.94" y2="317.5" width="0.1524" layer="91"/>
 <wire x1="408.94" y1="317.5" x2="386.08" y2="317.5" width="0.1524" layer="91"/>
-<pinref part="IO2" gate="G$1" pin="1"/>
 <wire x1="386.08" y1="317.5" x2="386.08" y2="315.976" width="0.1524" layer="91"/>
 </segment>
@@
 <label x="406.4" y="312.42" size="1.27" layer="95" rot="R180" xref="yes"/>
 <pinref part="R11" gate="G$1" pin="2"/>
-<pinref part="IO1" gate="G$1" pin="1"/>
 <wire x1="408.94" y1="312.42" x2="386.08" y2="312.42" width="0.1524" layer="91"/>
 <wire x1="386.08" y1="312.42" x2="386.08" y2="313.436" width="0.1524" layer="91"/>
@@
 <wire x1="429.26" y1="320.04" x2="408.94" y2="320.04" width="0.1524" layer="91"/>
 <pinref part="SUPPLY34" gate="G$1" pin="+5V"/>
-<wire x1="408.94" y1="320.04" x2="408.94" y2="327.66" width="0.1524" layer="91"/>
-<junction x="408.94" y="320.04"/>
-<pinref part="IO3" gate="G$1" pin="1"/>
-<wire x1="408.94" y1="327.66" x2="396.24" y2="327.66" width="0.1524" layer="91"/>
-<wire x1="396.24" y1="327.66" x2="396.24" y2="326.136" width="0.1524" layer="91"/>
 </segment>
 <segment>
@@
 <wire x1="459.74" y1="297.18" x2="459.74" y2="314.96" width="0.1524" layer="91"/>
 <junction x="459.74" y="314.96"/>
+<wire x1="480.06" y1="314.96" x2="497.84" y2="314.96" width="0.1524" layer="91"/>
+<pinref part="USB1_P" gate="G$1" pin="1"/>
 </segment>
 </net>
@@
 <wire x1="464.82" y1="292.1" x2="464.82" y2="312.42" width="0.1524" layer="91"/>
 <junction x="464.82" y="312.42"/>
+<wire x1="480.06" y1="312.42" x2="497.84" y2="312.42" width="0.1524" layer="91"/>
+<junction x="480.06" y="312.42"/>
+<pinref part="USB1_N" gate="G$1" pin="1"/>
 </segment>
 </net>
@@
 <pinref part="R36" gate="G$1" pin="2"/>
 <junction x="436.88" y="223.52"/>
-<pinref part="TH0" gate="G$1" pin="1"/>
-<wire x1="447.04" y1="238.76" x2="436.88" y2="238.76" width="0.1524" layer="91"/>
-<wire x1="436.88" y1="238.76" x2="436.88" y2="223.52" width="0.1524" layer="91"/>
 </segment>
 <segment>
@@
 <junction x="392.43" y="223.52"/>
 <junction x="398.78" y="223.52"/>
-<wire x1="373.38" y1="223.52" x2="392.43" y2="223.52" width="0.1524" layer="91"/>
+<wire x1="373.38" y1="223.52" x2="375.92" y2="223.52" width="0.1524" layer="91"/>
 <pinref part="J3" gate="A" pin="4"/>
-</segment>
-</net>
+<wire x1="375.92" y1="223.52" x2="392.43" y2="223.52" width="0.1524" layer="91"/>
+<wire x1="375.92" y1="223.52" x2="375.92" y2="228.6" width="0.1524" layer="91"/>
+<junction x="375.92" y="223.52"/>
+<wire x1="375.92" y1="228.6" x2="373.38" y2="228.6" width="0.1524" layer="91"/>
+<pinref part="TH0A" gate="G$1" pin="1"/>
+</segment>
+</net>
