File: Adithyas Design/FW_Toolboard1_v71(Eagle 9).brd (EAGLE design)
At the start: 54 x 40 mm, 151 parts, among them J2 2828XX-2282837-2, J3 430450400CON_430450400_MOL, M1 NMOSFET_WSD3066DN33, M2 CJ3400, M3 CJ3400, M4 CJ3400, P1 TPS54202_BUCKCONV, P2 3.3V, U1 RP2040IC57_RP2040-L, U2 W25Q128JVSIQSOIC_128JVSIQ_WIN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

Commit message: Routed most of the componenets to RP2040, Driver and GPIs remianing
Routing:
- net GND: vias 276 -> 275
