File: TD_Tool Board V2/TD_Tool Board V2/TD Toolboard V2.brd (EAGLE design)
At the start: 54.2 x 49 mm, 138 parts, among them J3 JST-MICROFIT, M1 NMOSFET_WSD3066DN33, M2 CJ3400, M3 CJ3400, M4 CJ3400, P1 TPS54202_BUCKCONV, P2 3.3V, U1 RP2040, U2 W25Q128, U3 SN65HVD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

Commit message: Fixed errors, Passed DRC, added logos
Parts:
- added U$1: (no value), FracktalWorks_Eagle_Library:FWLOGO_SMALL
- added U$2: (no value), FracktalWorks_Eagle_Library:MAKEININDIA
Other:
- board text added: "+"
- board text added: "-"
- board text added: "Dragon ToolBoard V2"
- board text added: "POWER"
Changed lines of the file:
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@@
 <text x="13.6144" y="33.3502" size="0.8128" layer="25" font="vector" ratio="15" rot="R180">CAN_H</text>
 <text x="8.636" y="19.6088" size="0.8128" layer="25" font="vector" ratio="15" rot="R270">+24</text>
-<text x="7.5438" y="24.1554" size="0.8128" layer="25" font="vector" ratio="15" rot="R270">GND</text>
+<text x="8.9408" y="23.5966" size="0.8128" layer="25" font="vector" ratio="15" rot="R270">GND</text>
 <text x="6.096" y="26.6192" size="0.508" layer="25" font="vector" ratio="15" rot="R270">+3.3V</text>
 <text x="5.8928" y="23.5458" size="0.508" layer="25" font="vector" ratio="15" rot="R270">+5V</text>
@@
 </text>
 <text x="5.8674" y="19.4056" size="0.508" layer="25" font="vector" ratio="15" rot="R270">+24V</text>
-<text x="56.6166" y="24.7142" size="0.508" layer="25" font="vector" ratio="15" rot="R270">A1</text>
-<text x="56.6928" y="22.0218" size="0.508" layer="25" font="vector" ratio="15" rot="R270">A2</text>
-<text x="56.6166" y="29.6418" size="0.508" layer="25" font="vector" ratio="15" rot="R270">B2</text>
-<text x="56.5912" y="27.1018" size="0.508" layer="25" font="vector" ratio="15" rot="R270">B1</text>
+<text x="58.7502" y="24.765" size="0.508" layer="25" font="vector" ratio="15" rot="R270">A1</text>
+<text x="58.7756" y="22.098" size="0.508" layer="25" font="vector" ratio="15" rot="R270">A2</text>
+<text x="58.674" y="29.6926" size="0.508" layer="25" font="vector" ratio="15" rot="R270">B2</text>
+<text x="58.6994" y="27.1272" size="0.508" layer="25" font="vector" ratio="15" rot="R270">B1</text>
 <text x="56.2356" y="40.7162" size="0.508" layer="25" font="vector" ratio="15" rot="R270">TH0</text>
 <text x="36.576" y="47.752" size="0.508" layer="25" font="vector" ratio="15" rot="R180">DN</text>
 <text x="34.671" y="48.0822" size="0.508" layer="25" font="vector" ratio="15" rot="R180">DP</text>
-<text x="57.3532" y="16.383" size="0.508" layer="25" font="vector" ratio="15" rot="R90">HE0</text>
+<text x="59.3344" y="16.5608" size="0.508" layer="25" font="vector" ratio="15" rot="R90">HE0</text>
+<text x="53.848" y="20.7518" size="0.8128" layer="25" rot="SR270">Dragon ToolBoard V2</text>
+<text x="11.6078" y="40.5384" size="0.8128" layer="25" font="vector">+</text>
+<text x="12.2174" y="45.6692" size="0.8128" layer="25" font="vector" rot="R90">-</text>
+<text x="12.2428" y="30.6578" size="0.8128" layer="25" font="vector" rot="R90">-</text>
+<text x="12.2428" y="25.5524" size="0.8128" layer="25" font="vector" rot="R90">+</text>
+<text x="11.5824" y="14.5796" size="0.8128" layer="26" font="vector" rot="MR90">+</text>
+<text x="17.3482" y="14.4526" size="0.8128" layer="26" font="vector" rot="MR0">-</text>
+<text x="25.4" y="14.5796" size="0.8128" layer="26" font="vector" rot="MR0">-</text>
+<text x="20.2692" y="14.478" size="0.8128" layer="26" font="vector" rot="MR0">+</text>
+<text x="40.0304" y="14.5542" size="0.8128" layer="26" font="vector" rot="MR0">+</text>
+<text x="45.1866" y="14.605" size="0.8128" layer="26" font="vector" rot="MR0">-</text>
+<text x="8.1026" y="19.8882" size="0.6096" layer="26" font="vector" ratio="15" rot="MR270">POWER</text>
 </plain>
 <attributes>
@@
 <attribute name="MANUFACTURER_PART_NUMBER" value="SN74LVC1G17DBVR" x="50.2666" y="24.2316" size="1.778" layer="27" rot="R180" display="off"/>
 <attribute name="MFR_NAME" value="Texas Instruments" x="50.2666" y="24.2316" size="1.778" layer="27" rot="R180" display="off"/>
-<attribute name="NAME" x="53.5378" y="17.2466" size="0.508" layer="27" font="vector" ratio="15" rot="R180"/>
+<attribute name="NAME" x="50.693" y="16.7132" size="0.508" layer="27" font="vector" ratio="15" rot="R180"/>
 <attribute name="VALUE" x="51.2588" y="18.923" size="0.508" layer="21" font="vector" ratio="15" rot="R180"/>
 </element>
@@
 <attribute name="MANUFACTURER" value="" x="25.8318" y="27.3304" size="1.778" layer="27" rot="R270" display="off"/>
 <attribute name="MPN" value="" x="25.8318" y="27.3304" size="1.778" layer="27" rot="R270" display="off"/>
-<attribute name="NAME" x="53.7728" y="17.1704" size="0.508" layer="25" font="vector" ratio="15" rot="R270" align="bottom-center"/>
+<attribute name="NAME" x="52.3758" y="17.1958" size="0.508" layer="25" font="vector" ratio="15" rot="R270" align="bottom-center"/>
 <attribute name="OPERATING_TEMP" value="" x="25.8318" y="27.3304" size="1.778" layer="27" rot="R270" display="off"/>
 <attribute name="PART_STATUS" value="" x="25.8318" y="27.3304" size="1.778" layer="27" rot="R270" display="off"/>
@@
 <attribute name="VALUE" x="45.7713" y="10.9665" size="0.508" layer="27" font="vector" ratio="15" rot="R180"/>
 </element>
+<element name="U$1" library="FracktalWorks_Eagle_Library" package="FWLOGO_SMALL" value="" x="53.6194" y="22.987" smashed="yes" rot="R270"/>
+<element name="U$2" library="FracktalWorks_Eagle_Library" package="MAKEININDIA" value="" x="55.5752" y="34.417" smashed="yes" rot="MR0"/>
 </elements>
 <signals>
@@
 <wire x1="55.9592" y1="35.817" x2="55.9592" y2="35.8394" width="0.2032" layer="1"/>
 <wire x1="50.9778" y1="31.3436" x2="54.1782" y2="34.544" width="0.2032" layer="16"/>
-<polygon width="0.1524" layer="1" pour="cutout">
-<vertex x="51.5512" y="5.3634"/>
-<vertex x="51.6512" y="5.3634" curve="90"/>
-</polygon>
 <via x="33.1978" y="34.8742" extent="1-16" drill="0.35"/>
 <via x="33.2232" y="35.687" extent="1-16" drill="0.35"/>
@@
 <wire x1="35.81914375" y1="31.512" x2="36.10014375" y2="31.231" width="0.2032" layer="1"/>
 <wire x1="31.87995625" y1="31.512" x2="35.81914375" y2="31.512" width="0.2032" layer="1"/>
-<wire x1="32.658" y1="33.4998" x2="34.0129" y2="33.4998" width="0.2032" layer="16"/>
-<wire x1="32.1112" y1="32.953" x2="32.658" y2="33.4998" width="0.2032" layer="16"/>
-<wire x1="34.0129" y1="33.4998" x2="35.179" y2="34.6659" width="0.2032" layer="16"/>
+<wire x1="32.658" y1="33.7284" x2="34.2415" y2="33.7284" width="0.2032" layer="16"/>
+<wire x1="32.658" y1="33.7284" x2="32.1112" y2="33.1816" width="0.2032" layer="16"/>
+<wire x1="32.1112" y1="32.953" x2="32.1112" y2="33.1816" width="0.2032" layer="16"/>
+<wire x1="34.2415" y1="33.7284" x2="35.179" y2="34.6659" width="0.2032" layer="16"/>
 <wire x1="35.179" y1="34.6659" x2="35.179" y2="37.2364" width="0.2032" layer="16"/>
 </signal>
@@
 <wire x1="36.449" y1="39.751" x2="35.7124" y2="39.0144" width="0.2032" layer="16"/>
 <wire x1="35.7124" y1="39.0144" x2="35.7124" y2="34.4678" width="0.2032" layer="16"/>
-<wire x1="35.7124" y1="34.4678" x2="34.1884" y2="32.9438" width="0.2032" layer="16"/>
-<wire x1="34.1884" y1="32.9438" x2="32.9184" y2="32.9438" width="0.2032" layer="16"/>
-<via x="32.9184" y="32.9438" extent="1-16" drill="0.35"/>
-<wire x1="32.9184" y1="32.1522" x2="32.9184" y2="32.9438" width="0.2032" layer="1"/>
+<wire x1="35.7124" y1="34.4678" x2="34.29" y2="33.0454" width="0.2032" layer="16"/>
+<wire x1="34.29" y1="33.0454" x2="32.9692" y2="33.0454" width="0.2032" layer="16"/>
+<wire x1="32.9692" y1="33.0454" x2="32.9184" y2="32.9946" width="0.2032" layer="16"/>
+<via x="32.9184" y="32.9946" extent="1-16" drill="0.35"/>
+<wire x1="32.9184" y1="32.1522" x2="32.9184" y2="32.9946" width="0.2032" layer="1"/>
 <wire x1="32.9108" y1="32.1446" x2="32.9184" y2="32.1522" width="0.2032" layer="1"/>
 </signal>
@@
 <wire x1="14.2134" y1="38.3794" x2="10.5156" y2="38.3794" width="0.4064" layer="1"/>
 <wire x1="10.5156" y1="38.3794" x2="9.9568" y2="37.8206" width="0.4064" layer="1"/>
-<wire x1="9.9568" y1="37.8206" x2="9.8298" y2="37.6936" width="0.3048" layer="1"/>
-<wire x1="9.8298" y1="37.6936" x2="9.8298" y2="36.83" width="0.3048" layer="1"/>
-<wire x1="9.8298" y1="36.83" x2="9.8298" y2="36.0934" width="0.3048" layer="1"/>
-<wire x1="11.2522" y1="34.671" x2="11.8872" y2="34.671" width="0.3048" layer="1"/>
-<wire x1="9.8298" y1="36.0934" x2="11.2522" y2="34.671" width="0.3048" layer="1"/>
+<wire x1="9.9568" y1="37.8206" x2="9.8298" y2="37.6936" width="0.4064" layer="1"/>
+<wire x1="9.8298" y1="37.6936" x2="9.8298" y2="36.83" width="0.4064" layer="1"/>
+<wire x1="9.8298" y1="36.83" x2="9.8298" y2="36.0934" width="0.4064" layer="1"/>
+<wire x1="11.2522" y1="34.671" x2="11.8872" y2="34.671" width="0.4064" layer="1"/>
+<wire x1="9.8298" y1="36.0934" x2="11.2522" y2="34.671" width="0.4064" layer="1"/>
 </signal>
 <signal name="CAN_P" class="2">
@@
 <contactref element="SJ3" pad="2"/>
 <contactref element="USB" pad="11"/>
-<wire x1="25.2354" y1="48.049" x2="25.2354" y2="48.577" width="0.508" layer="1"/>
-<wire x1="25.2354" y1="48.577" x2="24.9174" y2="48.895" width="0.508" layer="1"/>
-<wire x1="24.9174" y1="48.895" x2="24.9174" y2="49.7586" width="0.508" layer="1"/>
+<wire x1="25.2354" y1="48.049" x2="25.2354" y2="48.7548" width="0.508" layer="1"/>
+<wire x1="25.2354" y1="48.7548" x2="24.9174" y2="49.0728" width="0.508" layer="1"/>
+<wire x1="24.9174" y1="49.0728" x2="24.9174" y2="49.7586" width="0.508" layer="1"/>
 <wire x1="24.9174" y1="49.7586" x2="25.4254" y2="50.2666" width="0.508" layer="1"/>
 <wire x1="25.4254" y1="50.2666" x2="27.4574" y2="50.2666" width="0.508" layer="1"/>
