File: TD_Tool Board V3/TD_Tool Board V3/TD Toolboard V3.sch (EAGLE design)
At the start: 141 parts, among them J3 430450400CON_430450400_MOL, M1 NMOSFET_WSD3066DN33, M2 CJ3400, M3 CJ3400, M4 CJ3400, P1 TPS54202_BUCKCONV, P2 3.3V, U1 RP2040IC57_RP2040-L, U2 W25Q128JVSIQSOIC_128JVSIQ_WIN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, U3 SN65HVD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

Commit message: Made the required changes - renamed toolboard to V3
Parts:
- removed FD1, FD2, FD3: FIDUCIAL, CDC Library:FIDUCIAL
- removed X4: JST-XH-04-PIN-LONG-PAD, Rembrandt Electronics - JST XH Connectors v1-0:JST-XH-04-PIN-LONG-PAD
- added EXTRUDER: JST-XH-04-PIN-LONG-PAD, Rembrandt Electronics - JST XH Connectors v1-0:JST-XH-04-PIN-LONG-PAD
- C_FAN2: value JST-XH-02-PIN-LONG-PAD -> JST-XH
- D9: device LED:CHIP-FLAT-G_0603-0.35MM -> led:LED3MM
- J3: value 430450400CON_430450400_MOL -> JST-MICROFIT
- U1: value RP2040IC57_RP2040-L -> RP2040
- U2: value W25Q128JVSIQSOIC_128JVSIQ_WIN-L -> W25Q128
- U5: value ADXL345BCCZ-RL -> ADXL345
- U6: value SN74LVC1G17DBVRDBV5-L -> SN74L
- U7: value TMC2209-LA-TQFN28_5X5_3X8_EPAD_TRI -> TMC2209
- USB: value USB-C(DX07S016JA1R1500) -> USB-C(KH-TYPE-C-16P); device CDC Library:USB-C(DX07S016JA1R1500) -> Fracktal Misc Lib:USB-C(KH-TYPE-C-16P); DATASHEET (none) -> https://datasheet.lcsc.com/lcsc/2009111434_Shenzhen-Kinghel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; VENDOR (none) -> LCSC
- renumbered X2 to CANBUS, X3 to ENDSTOP, X5 to H_FAN, X6 to M_FAN, X7 to C_FAN, X8 to C_FAN2
Connections:
- removed net FAN1D: M3.D, M_FAN-1.S
- removed net N$2: C_FAN-1.S, C_FAN2-1.S, M4.D
- new net N$3: M3.D, M_FAN-2.S
- new net N$4: C_FAN-2.S, C_FAN2-2.S, M4.D
- net +24V: now also C_FAN-1.S, C_FAN2-1.S, H_FAN-1.S, M_FAN-1.S; no longer C_FAN-2.S, C_FAN2-2.S, H_FAN-2.S, M_FAN-2.S
- net A1: now also EXTRUDER-2.S; no longer X4-2.S
- net A2: now also EXTRUDER-1.S; no longer X4-1.S
- net B1: now also EXTRUDER-3.S; no longer X4-3.S
- net B2: now also EXTRUDER-4.S; no longer X4-4.S
- net N$1: now also H_FAN-2.S; no longer H_FAN-1.S
- net USB1_N: now also IO1.1
- net USB1_P: now also IO2.1
- net USB_N: no longer IO1.1
- net USB_P: no longer IO2.1
Other:
- moved on the sheet: A1, A2, B1, B2, IO1, IO2, USB
